File: Hardware/Project-TSC-PCB.brd (EAGLE design)
At the start: 46 x 35 mm, 105 parts, among them IC1 BQ25180YBGR_BQ25180YBGR, IC2 DRV2605YZFR_DRV2605YZFR, IC3 BMA423_BMA423, IC9 RT6160AWSC_RT6160AWSC, J1 503480-2400_503480-2400, J2 TC2030-IDC_TC2030-IDC, J4 KH-TYPE-C-16P_KH-TYPE-C-16P, Q1 20V/4.2A/52mΩ/1.4W, Q3 ESP32_C6_LIBRARY_6_SI1308EDL-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, U3 ESP32_C6_LIBRARY_MAX17048G+T10, X1 32MHz, X2 32.768kHz

Commit message: Hardware
Parts:
- removed R_PWE_EPD, R_PWE_EPD1, R_PWE_EPD2, R_PWE_EPD3: 10K, InkTime_v5:CPF0201D7K68C1_0201
- added R5, R7, R8, R_PWR_EPD: 10K, InkTime_v5:CPF0201D7K68C1_0201
- C1, C10, C11, C12, C13, C16, C17, C18, C2, C22, C3, C4, C5, C7, C8, C9, EPD_C5: device InkTime_v5:PERFECT_0402_0402 -> InkTime_v5:NORDIC_NRF_3_RESC0201_L
- C19: value 100uF -> 100nF
- moved R_TYPE_SEL 175.8 mm to (-10.2, -6.57), turned to 180 degrees
- moved EPD_C11 175.0 mm to (-15.2, -7.62), turned to 270 degrees
- moved Q3 173.3 mm to (-19.1, -9.75), turned to 180 degrees
- moved C25 169.8 mm to (-16.9, 11.4), turned to 90 degrees
- moved C39 161.9 mm to (-13.9, 9.73), turned to 270 degrees
- moved C33 161.4 mm to (-8.89, 8.89), turned to 90 degrees
- moved EPD_C1 160.8 mm to (-11.4, 2.44)
- moved EPD_C2 155.1 mm to (-11.4, 3.51)
- moved EPD_C6 154.7 mm to (-11.6, -3.44)
- moved EPD_C7 150.7 mm to (-11.6, -4.50)
- moved C10 149.2 mm to (4.70, 1.70)
- moved L5 147.5 mm to (-19.1, -13.8), turned to 180 degrees
- moved C13 147.2 mm to (1.27, 4.40), turned to 90 degrees
- moved EPD_C8 146.9 mm to (-11.6, -5.55)
- moved EPD_C9 143.7 mm to (-15.2, -3.81), turned to 90 degrees
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Connections:
- net 3V3: now also R5.2, R7.2, R8.2, R_PWR_EPD.2; no longer R_PWE_EPD.2, R_PWE_EPD1.2, R_PWE_EPD2.2, R_PWE_EPD3.2
- net EPD_3V3: now also EPD_C5.2; no longer EPD_C5.1
- net GND: now also C17.1, C18.1, EPD_C5.1; no longer C17.2, C18.2, EPD_C5.2
- net N$17: now also C17.2; no longer C17.1
- net N$18: now also C18.2; no longer C18.1
- net P0.13: now also R5.1; no longer R_PWE_EPD3.1
- net P0.14: now also R8.1; no longer R_PWE_EPD2.1
- net P1.01: now also R_PWR_EPD.1; no longer R_PWE_EPD.1
- net P1.02: now also R7.1; no longer R_PWE_EPD1.1
Routing:
- net GND: track 20.7 -> 256.0 mm, vias 2 -> 16
- net VBUS: track 0.00 -> 75.8 mm, vias 0 -> 4
- net SDA: track 0.00 -> 70.5 mm, vias 0 -> 5
- net 3V3: track 43.7 -> 112.0 mm, vias 4 -> 8
- net EPD_3V3: track 0.00 -> 59.1 mm, vias 0 -> 3
- net SCL: track 24.1 -> 81.1 mm, vias 2 -> 8
- net P1.02: track 0.00 -> 47.1 mm, vias 0 -> 4
- net ALERT: track 0.00 -> 43.1 mm, vias 0 -> 2
- net D-: track 0.00 -> 32.5 mm, vias 0 -> 2
- net HAPTIC_EN: track 0.00 -> 30.7 mm, vias 0 -> 2
- net IMU_INT1: track 0.00 -> 29.0 mm, vias 0 -> 2
- net D+: track 0.00 -> 23.4 mm, vias 0 -> 2
- net RESE: track 0.00 -> 22.5 mm, vias 0 -> 3
- net SCK: track 0.00 -> 22.2 mm, vias 0 -> 2
- net DEC4_6: track 0.00 -> 21.9 mm, vias 0 -> 2
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Other:
- board text added: "GND"
