File: Hardware/Project-TSC.sch (EAGLE design)
At the start: 105 parts, among them IC1 BQ25180YBGR_BQ25180YBGR, IC2 DRV2605YZFR_DRV2605YZFR, IC3 BMA423_BMA423, IC9 RT6160AWSC_RT6160AWSC, J1 503480-2400_503480-2400, J2 TC2030-IDC_TC2030-IDC, J4 KH-TYPE-C-16P_KH-TYPE-C-16P, Q1 20V/4.2A/52mΩ/1.4W, Q3 ESP32_C6_LIBRARY_6_SI1308EDL-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, U3 ESP32_C6_LIBRARY_MAX17048G+T10, X1 32MHz, X2 32.768kHz

Commit message: Hardware
Parts:
- C1, C10, C11, C12, C13, C16, C17, C18, C2, C22, C3, C4, C5, C7, C8, C9, EPD_C5: device InkTime_v5:PERFECT_0402_CAP_0402 -> InkTime_v5:NORDIC_NRF_3_CAPACITOR_0201_L
- C19: value 100uF -> 100nF
- renumbered R_PWE_EPD to R_PWR_EPD, R_PWE_EPD1 to R7, R_PWE_EPD2 to R8, R_PWE_EPD3 to R5
Connections:
- net EPD_3V3: now also EPD_C5.2; no longer EPD_C5.1
- net GND: now also C17.1, C18.1, EPD_C5.1; no longer C17.2, C18.2, EPD_C5.2
- net N$17: now also C17.2; no longer C17.1
- net N$18: now also C18.2; no longer C18.1
